File: i2s_rxtx.sch (KiCad schematic (older format))
At the start: 53 parts, among them IC1 AM26C32, IC2 AM26C31, IC3 AM26C31, J1 CONN_01x02, J2 RJ45_Shielded, J3 CONN_01x05, J4 RJ45_Shielded, J5 RJ45_Shielded

Commit message: adjusted pcb layout to new termination network
Parts:
- C10, C11, C12, C13, C14, C15, C16, C17, C18, C19, C20, C21: renamed from C?; footprint (none) -> Capacitor_SMD:C_0805_2012Metric_Pad1.15x1.40mm_HandSolder; symbol agg:C -> i2s_rxtx-rescue:C-agg
- C2, C3, C4, C5, C6, C7, C8, C9: symbol agg:C -> i2s_rxtx-rescue:C-agg
- FL1, FL2, FL3, FL4: renamed from FL?; footprint (none) -> agg:B82789_PinSwap
- IC1: symbol agg:AM26C32 -> i2s_rxtx-rescue:AM26C32-agg
- IC2, IC3: symbol agg:AM26C31 -> i2s_rxtx-rescue:AM26C31-agg
- J1: symbol agg:CONN_01x02 -> i2s_rxtx-rescue:CONN_01x02-agg
- J3: symbol agg:CONN_01x05 -> i2s_rxtx-rescue:CONN_01x05-agg
- R1: footprint Resistor_SMD:R_1206_3216Metric_Pad1.42x1.75mm_HandSolder -> Resistor_SMD:R_0805_2012Metric_Pad1.15x1.40mm_HandSolder; symbol agg:R -> i2s_rxtx-rescue:R-agg
- R10, R11, R12, R13, R14, R15, R16: renamed from R?; symbol agg:R -> i2s_rxtx-rescue:R-agg
- R2, R3, R4, R6, R7, R8, R9: renamed from R?; footprint Resistor_SMD:R_1206_3216Metric_Pad1.42x1.75mm_HandSolder -> Resistor_SMD:R_0805_2012Metric_Pad1.15x1.40mm_HandSolder; symbol agg:R -> i2s_rxtx-rescue:R-agg
- R5: symbol agg:R -> i2s_rxtx-rescue:R-agg
